File: hardware/R2XXX_logger/FPGA.kicad_sch (KiCad schematic)
At the start: 1 part, among them U2 ICE40UP5K-SG48ITR

Commit message: Throws flatbuf packets
Parts:
- renumbered U2 to U4
Changed lines of the file:
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@@
 		(dnp no)
 		(fields_autoplaced yes)
-		(property "Reference" "U2"
+		(property "Reference" "U4"
 			(at 115.57 81.2799 0)
 			(show_name no)
@@
 			(project "R2XXX_logger"
 				(path "/77c40bdb-f224-4f9c-bece-a146e46e73be/3647f277-d804-4cc5-a736-cb9e0e2670ce"
-					(reference "U2")
+					(reference "U4")
 					(unit 1)
 				)
@@
 		(dnp no)
 		(fields_autoplaced yes)
-		(property "Reference" "U2"
+		(property "Reference" "U4"
 			(at 125.73 148.5899 0)
 			(show_name no)
@@
 			(project "R2XXX_logger"
 				(path "/77c40bdb-f224-4f9c-bece-a146e46e73be/3647f277-d804-4cc5-a736-cb9e0e2670ce"
-					(reference "U2")
+					(reference "U4")
 					(unit 4)
 				)
@@
 		(dnp no)
 		(fields_autoplaced yes)
-		(property "Reference" "U2"
+		(property "Reference" "U4"
 			(at 152.4 142.24 0)
 			(show_name no)
@@
 			(project "R2XXX_logger"
 				(path "/77c40bdb-f224-4f9c-bece-a146e46e73be/3647f277-d804-4cc5-a736-cb9e0e2670ce"
-					(reference "U2")
+					(reference "U4")
 					(unit 2)
 				)
@@
 		(dnp no)
 		(fields_autoplaced yes)
-		(property "Reference" "U2"
+		(property "Reference" "U4"
 			(at 95.25 128.2699 0)
 			(show_name no)
@@
 			(project "R2XXX_logger"
 				(path "/77c40bdb-f224-4f9c-bece-a146e46e73be/3647f277-d804-4cc5-a736-cb9e0e2670ce"
-					(reference "U2")
+					(reference "U4")
 					(unit 3)
 				)
